File: PCB/anemometer.kicad_sch (KiCad schematic)
At the start: 16 parts

Commit message: WIP - PCB
Parts:
- added C? (x2): 0.1µF, symbol Device:C
- added C?: 1µF, symbol Device:C
- added LS?: US_W, symbol Device:Speaker_Ultrasound
- added LS?: US_C, symbol Device:Speaker_Ultrasound
- added R?: 1k, symbol Device:R
- added R?: 10k, symbol Device:R
- added U?: 4046, symbol 4xxx:4046
- R?: value 1k -> 10k
Connections:
- net GND: now also LS?.2, U?.8 (VSS)
- net VDD: now also R?.1, U?.16 (VDD)
- net at Q?.3 (C): now also C?.2, R?.2
- net at R?.2, U?.3 (RefIn), U?.4 (FOUT): now also U?.3 (RefIn)
- new net: C?.1, LS?.1 (x2)
- new net: R?.1, U?.2 (PC1)
- new net US_PD1: C?.1, R?.2
Other:
- note added: "Hierarchical Pins"
- moved on the sheet: C?, R?
