File: Anemo/anemometer.kicad_sch (KiCad schematic)
At the start: 24 parts

Commit message: Anemo PCB
Parts:
- removed J?: Conn_01x05_Male, Connector_PinHeader_2.54mm:PinHeader_1x05_P2.54mm_Vertical, symbol Connector:Conn_01x05_Male
- removed LS?: US_E, symbol Device:Speaker_Ultrasound
- removed LS?: US_N, symbol Device:Speaker_Ultrasound
- removed LS?: US_C, symbol Device:Speaker_Ultrasound
- removed LS?: US_W, symbol Device:Speaker_Ultrasound
- added C7: 0.1µF, Capacitor_THT:C_Disc_D5.0mm_W2.5mm_P5.00mm, symbol Device:C
- added C8: 1µF, Capacitor_THT:C_Disc_D5.0mm_W2.5mm_P5.00mm, symbol Device:C
- added J1: Conn_01x04_Male, Connector_PinHeader_2.54mm:PinHeader_1x04_P2.54mm_Vertical, symbol Connector:Conn_01x04_Male
- added LS4: US_E, Buzzer_Beeper:Buzzer_D14mm_H7mm_P10mm, symbol Device:Speaker_Ultrasound
- added R8: 10k, Resistor_SMD:R_0805_2012Metric_Pad1.20x1.40mm_HandSolder, symbol Device:R
- added U3: 4046, Package_DIP:DIP-16_W7.62mm_Socket_LongPads, symbol 4xxx:4046
- C1, C2, C3, C4, C5, C6: renamed from C?; footprint (none) -> Capacitor_THT:C_Disc_D5.0mm_W2.5mm_P5.00mm
- LS1, LS2, LS3: renamed from LS?; footprint (none) -> Buzzer_Beeper:Buzzer_D14mm_H7mm_P10mm
- R1: renamed from R?; value 10k -> (none)
- R2, R3, R4, R5, R6, R7: renamed from R?; footprint (none) -> Resistor_SMD:R_0805_2012Metric_Pad1.20x1.40mm_HandSolder
- U1, U2: renamed from U?; footprint (none) -> Package_DIP:DIP-16_W7.62mm_Socket_LongPads
- gave numbers to parts that had none: 1
Connections:
- net GND: now also C6.2, LS3.2, C8.2, J1.1 (Pin_1), LS4.2, U3.8 (VSS)
- net VDD: now also J1.2 (Pin_2), U3.16 (VDD)
- net at C5.2: now also U2.14 (SigIn)
- net at R5.2, U1.3 (RefIn), U1.4 (FOUT)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: now also U3.3 (RefIn)
- net US_PD1 renamed US_PD_WEST
- net US_PD_WEST: now also J1.4 (Pin_4)
- new net: C7.2, U3.14 (SigIn)
- new net: R8.1, U3.2 (PC1)
- new net: C7.1, LS4.1
- new net US_PD_EAST: C8.1, J1.3 (Pin_3), R8.2
Other:
- note added: "Pins"
- note removed: "Hierarchical Pins"
- moved on the sheet: C1, C2, C3, C4, C5, C6, LS1, LS2, LS3, Q1, R1, R2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
